File: Electronics/Debug_adapter.brd (EAGLE design)
At the start: 38.4 x 22.9 mm, 12 parts, among them X1 USBSMD

Commit message: updated ground connection in debug adapter
Connections:
- removed net N$6: JP1.10, JP1.2, U$1.P$10, U$2.P$2, U$3.P$3
- net GND: now also JP1.10, JP1.2, U$1.P$10, U$2.P$2, U$3.P$3
Routing:
- net GND: track 27.9 -> 82.9 mm
- net N$6: track 49.6 -> 0.00 mm
Changed lines of the file:
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@@
 <via x="30.988" y="10.414" extent="1-16" drill="0.6096"/>
-</signal>
-<signal name="N$6">
-<contactref element="JP1" pad="10"/>
-<contactref element="U$1" pad="P$10"/>
-<contactref element="JP1" pad="2"/>
-<contactref element="U$2" pad="P$2"/>
-<contactref element="U$3" pad="P$3"/>
-<wire x1="9.906" y1="5.334" x2="12.065" y2="3.175" width="0.254" layer="16"/>
-<wire x1="5.08" y1="5.334" x2="9.906" y2="5.334" width="0.254" layer="16"/>
-<wire x1="3.048" y1="3.302" x2="5.08" y2="5.334" width="0.254" layer="16"/>
-<wire x1="3.048" y1="3.302" x2="3.175" y2="3.175" width="0.254" layer="16"/>
-<wire x1="29.718" y1="17.272" x2="33.528" y2="17.272" width="0.254" layer="1"/>
-<wire x1="29.718" y1="13.716" x2="29.718" y2="17.272" width="0.254" layer="1"/>
-<wire x1="28.702" y1="12.7" x2="29.718" y2="13.716" width="0.254" layer="1"/>
-<wire x1="33.528" y1="17.272" x2="33.67" y2="17.38" width="0.254" layer="1"/>
-<wire x1="28.702" y1="12.7" x2="28.575" y2="12.7" width="0.254" layer="1"/>
-<wire x1="29.718" y1="3.556" x2="28.702" y2="2.54" width="0.254" layer="1"/>
-<wire x1="29.718" y1="13.716" x2="29.718" y2="3.556" width="0.254" layer="1"/>
-<wire x1="28.702" y1="2.54" x2="28.575" y2="2.54" width="0.254" layer="1"/>
-<wire x1="13.97" y1="1.27" x2="12.065" y2="3.175" width="0.254" layer="16"/>
-<wire x1="27.178" y1="1.27" x2="13.97" y2="1.27" width="0.254" layer="16"/>
-<wire x1="28.448" y1="2.54" x2="27.178" y2="1.27" width="0.254" layer="16"/>
-<wire x1="28.448" y1="2.54" x2="28.575" y2="2.54" width="0.254" layer="16"/>
 </signal>
 <signal name="N$7">
@@
 <via x="11.43" y="10.16" extent="1-16" drill="0.6096"/>
 <via x="16.002" y="11.938" extent="1-16" drill="0.6096"/>
+<contactref element="JP1" pad="10"/>
+<contactref element="U$1" pad="P$10"/>
+<contactref element="JP1" pad="2"/>
+<contactref element="U$2" pad="P$2"/>
+<contactref element="U$3" pad="P$3"/>
+<wire x1="9.906" y1="5.334" x2="12.065" y2="3.175" width="0.254" layer="16"/>
+<wire x1="5.08" y1="5.334" x2="9.906" y2="5.334" width="0.254" layer="16"/>
+<wire x1="3.048" y1="3.302" x2="5.08" y2="5.334" width="0.254" layer="16"/>
+<wire x1="3.048" y1="3.302" x2="3.175" y2="3.175" width="0.254" layer="16"/>
+<wire x1="29.718" y1="17.272" x2="33.528" y2="17.272" width="0.254" layer="1"/>
+<wire x1="29.718" y1="13.716" x2="29.718" y2="17.272" width="0.254" layer="1"/>
+<wire x1="28.702" y1="12.7" x2="29.718" y2="13.716" width="0.254" layer="1"/>
+<wire x1="33.528" y1="17.272" x2="33.67" y2="17.38" width="0.254" layer="1"/>
+<wire x1="28.702" y1="12.7" x2="28.575" y2="12.7" width="0.254" layer="1"/>
+<wire x1="29.718" y1="3.556" x2="28.702" y2="2.54" width="0.254" layer="1"/>
+<wire x1="29.718" y1="13.716" x2="29.718" y2="3.556" width="0.254" layer="1"/>
+<wire x1="28.702" y1="2.54" x2="28.575" y2="2.54" width="0.254" layer="1"/>
+<wire x1="13.97" y1="1.27" x2="12.065" y2="3.175" width="0.254" layer="16"/>
+<wire x1="27.178" y1="1.27" x2="13.97" y2="1.27" width="0.254" layer="16"/>
+<wire x1="28.448" y1="2.54" x2="27.178" y2="1.27" width="0.254" layer="16"/>
+<wire x1="28.448" y1="2.54" x2="28.575" y2="2.54" width="0.254" layer="16"/>
+<wire x1="11.43" y1="10.16" x2="11.43" y2="6.858" width="0.4064" layer="16"/>
+<wire x1="11.43" y1="6.858" x2="9.906" y2="5.334" width="0.4064" layer="16"/>
 </signal>
 <signal name="N$13">
