File: Electronics/Maveric32_autopilot/Rev4.1.1/MegaFly_rev4.1.1.sch (EAGLE design)
At the start: 115 parts, among them J1 SOLDER_JUMPER_2WAY, J2 SOLDER_JUMPER_2WAY, J3 SOLDER_JUMPER_2WAY, P1 POWER, P10 POWERSMALL_SMD, P11 POWERSMALL_SMD, P12 POWERSMALL_SMD, P13 POWERSMALL_SMD, P2 AVR32_JTAG+SERIALMOLEX_PICOBL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, P5 SPEKTRUM_RECEIVER, P6 SPEKTRUM_RECEIVER, P8 SENSOR, P9 SENSOR, Q1 N-CHANNEL_SOT23, Q2 N-CHANNEL_SOT23, Q3 N-CHANNEL_SOT23, Q4 N-CHANNEL_SOT23, Q5 MOSFET-PCHANNELSMD, U1 LM2734, U10 AT32UC3C1512/1256/1128, U2 MC78L05, U3 V_REG_MIC5235-3.3, U4 LM2734, U50 BMP180, U60 HMC5883L, U70 LSM330DLC, X1 CRYSTAL:ABM_16MHz

Commit message: Update Electronics files: sch, brd and xls with new component references
Parts:
- R2: DISTRIBUTOR (none) -> Digikey; ORDER_CODE (none) -> RMCF0603FT31K6CT-ND
- R24: DISTRIBUTOR (none) -> Digikey; ORDER_CODE (none) -> PNM0603-25KBCT-ND
- R9: DISTRIBUTOR (none) -> Digikey; ORDER_CODE (none) -> 311-.25SCT-ND
Changed lines of the file:
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@@
 <grid distance="0.1" unitdist="inch" unit="inch" style="lines" multiple="1" display="no" altdistance="0.01" altunitdist="inch" altunit="inch"/>
 <layers>
-<layer number="1" name="Top" color="12" fill="1" visible="yes" active="no"/>
-<layer number="16" name="Bottom" color="9" fill="1" visible="yes" active="no"/>
-<layer number="17" name="Pads" color="2" fill="1" visible="yes" active="no"/>
-<layer number="18" name="Vias" color="2" fill="1" visible="yes" active="no"/>
-<layer number="19" name="Unrouted" color="6" fill="1" visible="yes" active="no"/>
-<layer number="20" name="Dimension" color="15" fill="1" visible="yes" active="no"/>
-<layer number="21" name="tPlace" color="7" fill="1" visible="yes" active="no"/>
-<layer number="22" name="bPlace" color="7" fill="1" visible="yes" active="no"/>
-<layer number="23" name="tOrigins" color="15" fill="1" visible="yes" active="no"/>
-<layer number="24" name="bOrigins" color="15" fill="1" visible="yes" active="no"/>
-<layer number="25" name="tNames" color="15" fill="1" visible="yes" active="no"/>
-<layer number="26" name="bNames" color="15" fill="1" visible="yes" active="no"/>
-<layer number="27" name="tValues" color="7" fill="1" visible="yes" active="no"/>
-<layer number="28" name="bValues" color="7" fill="1" visible="yes" active="no"/>
+<layer number="1" name="Top" color="12" fill="1" visible="no" active="no"/>
+<layer number="16" name="Bottom" color="9" fill="1" visible="no" active="no"/>
+<layer number="17" name="Pads" color="2" fill="1" visible="no" active="no"/>
+<layer number="18" name="Vias" color="2" fill="1" visible="no" active="no"/>
+<layer number="19" name="Unrouted" color="6" fill="1" visible="no" active="no"/>
+<layer number="20" name="Dimension" color="15" fill="1" visible="no" active="no"/>
+<layer number="21" name="tPlace" color="7" fill="1" visible="no" active="no"/>
+<layer number="22" name="bPlace" color="7" fill="1" visible="no" active="no"/>
+<layer number="23" name="tOrigins" color="15" fill="1" visible="no" active="no"/>
+<layer number="24" name="bOrigins" color="15" fill="1" visible="no" active="no"/>
+<layer number="25" name="tNames" color="15" fill="1" visible="no" active="no"/>
+<layer number="26" name="bNames" color="15" fill="1" visible="no" active="no"/>
+<layer number="27" name="tValues" color="7" fill="1" visible="no" active="no"/>
+<layer number="28" name="bValues" color="7" fill="1" visible="no" active="no"/>
 <layer number="29" name="tStop" color="7" fill="3" visible="no" active="no"/>
 <layer number="30" name="bStop" color="7" fill="6" visible="no" active="no"/>
@@
 <layer number="35" name="tGlue" color="7" fill="4" visible="no" active="no"/>
 <layer number="36" name="bGlue" color="7" fill="5" visible="no" active="no"/>
-<layer number="37" name="tTest" color="7" fill="1" visible="yes" active="no"/>
-<layer number="38" name="bTest" color="7" fill="1" visible="yes" active="no"/>
+<layer number="37" name="tTest" color="7" fill="1" visible="no" active="no"/>
+<layer number="38" name="bTest" color="7" fill="1" visible="no" active="no"/>
 <layer number="39" name="tKeepout" color="4" fill="11" visible="no" active="no"/>
 <layer number="40" name="bKeepout" color="1" fill="11" visible="no" active="no"/>
@@
 <layer number="44" name="Drills" color="7" fill="1" visible="no" active="no"/>
 <layer number="45" name="Holes" color="7" fill="1" visible="no" active="no"/>
-<layer number="46" name="Milling" color="3" fill="1" visible="yes" active="no"/>
-<layer number="47" name="Measures" color="7" fill="1" visible="yes" active="no"/>
-<layer number="48" name="Document" color="7" fill="1" visible="yes" active="no"/>
-<layer number="49" name="Reference" color="7" fill="1" visible="yes" active="no"/>
-<layer number="50" name="dxf" color="7" fill="1" visible="yes" active="no"/>
-<layer number="51" name="tDocu" color="7" fill="1" visible="yes" active="no"/>
-<layer number="52" name="bDocu" color="7" fill="1" visible="yes" active="no"/>
-<layer number="53" name="tGND_GNDA" color="7" fill="9" visible="yes" active="no"/>
-<layer number="54" name="bGND_GNDA" color="1" fill="9" visible="yes" active="no"/>
-<layer number="56" name="wert" color="7" fill="1" visible="yes" active="no"/>
+<layer number="46" name="Milling" color="3" fill="1" visible="no" active="no"/>
+<layer number="47" name="Measures" color="7" fill="1" visible="no" active="no"/>
+<layer number="48" name="Document" color="7" fill="1" visible="no" active="no"/>
+<layer number="49" name="Reference" color="7" fill="1" visible="no" active="no"/>
+<layer number="50" name="dxf" color="7" fill="1" visible="no" active="no"/>
+<layer number="51" name="tDocu" color="7" fill="1" visible="no" active="no"/>
+<layer number="52" name="bDocu" color="7" fill="1" visible="no" active="no"/>
+<layer number="53" name="tGND_GNDA" color="7" fill="9" visible="no" active="no"/>
+<layer number="54" name="bGND_GNDA" color="1" fill="9" visible="no" active="no"/>
+<layer number="56" name="wert" color="7" fill="1" visible="no" active="no"/>
 <layer number="91" name="Nets" color="2" fill="1" visible="yes" active="yes"/>
 <layer number="92" name="Busses" color="1" fill="1" visible="yes" active="yes"/>
@@
 <part name="GND16" library="supply1" deviceset="GND" device=""/>
 <part name="R2" library="rcl" deviceset="R-EU_" device="R0603" value="31.6k">
-<attribute name="DISTRIBUTOR" value=""/>
-<attribute name="ORDER_CODE" value=""/>
+<attribute name="DISTRIBUTOR" value="Digikey"/>
+<attribute name="ORDER_CODE" value="RMCF0603FT31K6CT-ND"/>
 <attribute name="PLACE_PART" value="YES"/>
 </part>
@@
 </part>
 <part name="R9" library="rcl" deviceset="R-EU_" device="R0805" value="0.25R">
-<attribute name="DISTRIBUTOR" value=""/>
-<attribute name="ORDER_CODE" value=""/>
+<attribute name="DISTRIBUTOR" value="Digikey"/>
+<attribute name="ORDER_CODE" value="311-.25SCT-ND"/>
 <attribute name="PLACE_PART" value="YES"/>
 </part>
@@
 </part>
 <part name="R24" library="rcl" deviceset="R-EU_" device="R0603" value="25k">
-<attribute name="DISTRIBUTOR" value=""/>
-<attribute name="ORDER_CODE" value=""/>
+<attribute name="DISTRIBUTOR" value="Digikey"/>
+<attribute name="ORDER_CODE" value="PNM0603-25KBCT-ND"/>
 <attribute name="PLACE_PART" value="YES"/>
 </part>
@@
 <instance part="GND16" gate="1" x="-109.22" y="7.62"/>
 <instance part="R2" gate="G$1" x="-93.98" y="20.32" rot="R180">
-<attribute name="DISTRIBUTOR" x="-93.98" y="20.32" size="1.778" layer="96"/>
-<attribute name="ORDER_CODE" x="-93.98" y="20.32" size="1.778" layer="96"/>
+<attribute name="DISTRIBUTOR" x="-93.98" y="20.32" size="1.778" layer="96" display="off"/>
+<attribute name="ORDER_CODE" x="-93.98" y="20.32" size="1.778" layer="96" display="off"/>
 <attribute name="PLACE_PART" x="-93.98" y="20.32" size="1.778" layer="96" display="off"/>
 </instance>
@@
 </instance>
 <instance part="R24" gate="G$1" x="264.16" y="170.18" rot="R180">
-<attribute name="DISTRIBUTOR" x="264.16" y="170.18" size="1.778" layer="96"/>
-<attribute name="ORDER_CODE" x="264.16" y="170.18" size="1.778" layer="96"/>
+<attribute name="DISTRIBUTOR" x="264.16" y="170.18" size="1.778" layer="96" display="off"/>
+<attribute name="ORDER_CODE" x="264.16" y="170.18" size="1.778" layer="96" display="off"/>
 <attribute name="PLACE_PART" x="264.16" y="170.18" size="1.778" layer="96" display="off"/>
 </instance>

Commit message: Update DFU instructions and Add the polarity of SOT1 in electronics
Parts:
- LD1: ORDER_CODE (none) -> 754-1131-1-ND
Changed lines of the file:
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@@
 </part>
 <part name="LD1" library="LEDs" deviceset="LED" device="CHIPLED_0805_GREEN" value="green">
+<attribute name="ORDER_CODE" value="754-1131-1-ND"/>
 <attribute name="PLACE_PART" value="YES"/>
 <attribute name="UNIT_PRICE" value="0.25"/>

Commit message: Update wiki and electronics documentation
Connections:
- new net +5V: C5.2, D6.A, J1.P$2, J3.P$2, L2.2, R7.1
- net +6V: no longer C5.2, D6.A, J1.P$2, J3.P$2, L2.2, R7.1

Commit message: Revert "Update wiki and electronics documentation"
This reverts commit 820a4100233712abf54084fecef851c241c0b9cc.
Connections:
- removed net +5V: C5.2, D6.A, J1.P$2, J3.P$2, L2.2, R7.1
- net +6V: now also C5.2, D6.A, J1.P$2, J3.P$2, L2.2, R7.1
